File: 2/obd25k80.brd (EAGLE design)
At the start: 96.5 x 50.8 mm, 56 parts, among them IC1 PIC18F25K80, IC2 MCP2562, IC3 78L05, IC4 78L05, IC5 LE33CZ, J1 MA04-1, J2 DB9-M, Q1 BC547, Q2 BC557, Q3 BC547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

Commit message: Cleanup
Connections:
- net RA5 renamed C2INB
Changed lines of the file:
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@@
 <wire x1="36.83" y1="19.939" x2="36.83" y2="20.32" width="0.254" layer="16"/>
 </signal>
-<signal name="RA5">
+<signal name="C2INB">
 <contactref element="IC1" pad="7"/>
 <contactref element="R8" pad="2"/>
